Commit message: joy node with wrench transform

File: gazebo_test/robots/quad.urdf (robot description, URDF)
Before this commit: robot quad, 2 links, 1 joints
Links:
- link quad: mass None -> 0.8; geometry collision box size=0.4 0.4 0.1; visual cylinder length=0.1 radius=0.2

File: gazebo_test/urdf/quad.urdf.xacro (robot description, xacro)
@@ -7,5 +7,9 @@
   <link name="base_link" />
   <link name="quad">
-    <xacro:cylinder_inertia_def radius="0.2" length="0.1" mass="0.8" />
+    <inertial>
+      <origin xyz="0 0 0" rpy="0 0 0"/>
+      <mass value="0.8"/>
+      <xacro:cylinder_inertia_def radius="0.2" length="0.1" mass="0.8" />
+    </inertial>
     <visual>
       <geometry>
@@ -15,5 +19,5 @@
     <collision>
       <geometry>
-        <cylinder radius="0.2" length="0.1" />
+        <box size="0.4 0.4 0.1" />
       </geometry>
     </collision>
@@ -21,5 +25,5 @@
   <joint
     name="base_fixed_joint"
-    type="floating">
+    type="fixed">
     <origin
       xyz="0 0 0"
@@ -37,9 +41,4 @@
     <mu2>0.2</mu2>
   </gazebo>
-  <gazebo reference="base_link">
-    <material>Gazebo/Grey</material>
-    <mu1>0.2</mu1>
-    <mu2>0.2</mu2>
-  </gazebo>
   <gazebo>
     <plugin name="quad_controller" filename="libgazebo_ros_quad.so">
