Commit message: Gazebo related launchfiles and config

File: gazebo_test/urdf/quad.urdf.xacro (robot description, xacro)
@@ -21,5 +21,5 @@
   <joint
     name="base_fixed_joint"
-    type="fixed">
+    type="floating">
     <origin
       xyz="0 0 0"
@@ -29,6 +29,13 @@
     <parent
       link="base_link" />
+    <axis
+      xyz="0 0 0" />
   </joint>
   <gazebo reference="quad">
+    <material>Gazebo/Grey</material>
+    <mu1>0.2</mu1>
+    <mu2>0.2</mu2>
+  </gazebo>
+  <gazebo reference="base_link">
     <material>Gazebo/Grey</material>
     <mu1>0.2</mu1>

Commit message: drone mesh, relative force

File: gazebo_test/urdf/quad.urdf.xacro (robot description, xacro)
@@ -5,4 +5,7 @@
   <xacro:include filename="$(find gazebo_test)/urdf/common.xacro" />
   <xacro:include filename="$(find gazebo_test)/urdf/gazebo.urdf.xacro" />
+  <material name="Grey1">
+    <color rgba="0.1 0.1 0.1 1" />
+  </material>
   <link name="base_link" />
   <link name="quad">
@@ -13,7 +16,12 @@
     </inertial>
     <visual>
+      <origin
+        xyz="0 0 0.03"
+        rpy="0 0 0" />
       <geometry>
-        <cylinder radius="0.2" length="0.1" />
+        <mesh
+          filename="package://gazebo_test/meshes/quad.stl" />
       </geometry>
+      <material name="Grey1" />
     </visual>
     <collision>
